Commit message: 修复编译警告和SLAM节点启动问题
- 修复sensor_interface中未使用变量publish_rate的警告
- 优化setup_ros_env.sh，改进conda库路径清理逻辑
- 修复navigation.launch.py：sync_slam_toolbox_node不需要lifecycle_manager
- 更新URDF文件（robot_base.xacro和robot_gazebo.xacro）
- 添加TROUBLESHOOTING.md故障排除文档

File: src/vacuum_robot_sim/urdf/robot_base.xacro (robot description, xacro)
@@ -1,5 +1,4 @@
 <?xml version="1.0"?>
 <robot xmlns:xacro="http://www.ros.org/wiki/xacro" name="vacuum_robot">
-  <!-- 定义机器人参数 -->
   <xacro:property name="base_radius" value="0.18"/>
   <xacro:property name="base_height" value="0.1"/>
@@ -8,5 +7,7 @@
   <xacro:property name="base_mass" value="5.0"/>
   <xacro:property name="wheel_mass" value="0.5"/>
-  <!-- 基础链接 -->
+  <xacro:property name="caster_radius" value="0.015"/>
+  <xacro:property name="caster_mass" value="0.1"/>
+  <xacro:property name="caster_z_offset" value="${-1 * (base_height/2 + 2*wheel_radius - caster_radius) + 0.002}"/>
   <link name="base_link">
     <visual>
@@ -30,5 +31,4 @@
     </inertial>
   </link>
-  <!-- 左轮 -->
   <link name="left_wheel">
     <visual>
@@ -44,5 +44,5 @@
       <origin xyz="0 0 0" rpy="1.5708 0 0"/>
       <geometry>
-        <cylinder radius="${wheel_radius}" length="${wheel_width}"/>
+        <sphere radius="${wheel_radius}" length="${wheel_width}"/>
       </geometry>
     </collision>
@@ -52,5 +52,4 @@
     </inertial>
   </link>
-  <!-- 右轮 -->
   <link name="right_wheel">
     <visual>
@@ -66,5 +65,5 @@
       <origin xyz="0 0 0" rpy="1.5708 0 0"/>
       <geometry>
-        <cylinder radius="${wheel_radius}" length="${wheel_width}"/>
+        <sphere radius="${wheel_radius}" length="${wheel_width}"/>
       </geometry>
     </collision>
@@ -74,5 +73,4 @@
     </inertial>
   </link>
-  <!-- 左轮关节 -->
   <joint name="left_wheel_joint" type="continuous">
     <parent link="base_link"/>
@@ -81,12 +79,10 @@
     <axis xyz="0 1 0"/>
   </joint>
-  <!-- 右轮关节 -->
   <joint name="right_wheel_joint" type="continuous">
     <parent link="base_link"/>
     <child link="right_wheel"/>
-    <origin xyz="0 -${base_radius - wheel_width/2} -${base_height/2 + wheel_radius}" rpy="0 0 0"/>
+    <origin xyz="0 -${base_radius + wheel_width/2} -${base_height/2 + wheel_radius}" rpy="0 0 0"/>
     <axis xyz="0 1 0"/>
   </joint>
-  <!-- 激光雷达安装位置 -->
   <link name="laser_link">
     <visual>
@@ -105,3 +101,47 @@
     <origin xyz="${base_radius} 0 ${base_height/2}" rpy="0 0 0"/>
   </joint>
+  <link name="imu_link">
+    <visual>
+      <origin xyz="0 0 0" rpy="0 0 0"/>
+      <geometry>
+        <box size="0.03 0.03 0.01"/>
+      </geometry>
+      <material name="green">
+        <color rgba="0 1 0 1"/>
+      </material>
+    </visual>
+  </link>
+  <joint name="imu_joint" type="fixed">
+    <parent link="base_link"/>
+    <child link="imu_link"/>
+    <origin xyz="0 0 ${base_height/2}" rpy="0 0 0"/>
+  </joint>
+  <xacro:macro name="caster_xacro" params="prefix x_reflect">
+    <link name="${prefix}_caster">
+      <visual>
+        <geometry>
+          <sphere radius="${caster_radius}"/>
+        </geometry>
+        <material name="grey">
+          <color rgba="0.5 0.5 0.5 1"/>
+        </material>
+      </visual>
+      <collision>
+        <geometry>
+          <sphere radius="${caster_radius}"/>
+        </geometry>
+      </collision>
+      <inertial>
+        <mass value="${caster_mass}"/>
+        <inertia ixx="0.0001" ixy="0" ixz="0" iyy="0.0001" iyz="0" izz="0.0001"/>
+      </inertial>
+    </link>
+    <joint name="${prefix}_caster_joint" type="fixed">
+      <parent link="base_link"/>
+      <child link="${prefix}_caster"/>
+      <origin xyz="${x_reflect * 0.15} 0 ${caster_z_offset}" rpy="0 0 0"/>
+    </joint>
+  </xacro:macro>
+  <xacro:caster_xacro prefix="front" x_reflect="1.0"/>
+  <xacro:caster_xacro prefix="rear" x_reflect="-1.0"/>
 </robot>

File: src/vacuum_robot_sim/urdf/robot_gazebo.xacro (robot description, xacro)
@@ -2,5 +2,4 @@
 <robot xmlns:xacro="http://www.ros.org/wiki/xacro" name="vacuum_robot">
   <xacro:include filename="$(find vacuum_robot_sim)/urdf/robot_base.xacro"/>
-  <!-- Gazebo插件：差分驱动控制器 -->
   <gazebo>
     <plugin name="differential_drive_controller" filename="libgazebo_ros_diff_drive.so">
@@ -8,14 +7,10 @@
         <namespace>/</namespace>
       </ros>
-      <!-- 轮子设置 -->
       <left_joint>left_wheel_joint</left_joint>
       <right_joint>right_wheel_joint</right_joint>
-      <!-- 运动学特性 -->
-      <wheel_separation>${2 * base_radius}</wheel_separation>
+      <wheel_separation>${2 * (base_radius + wheel_width/2)}</wheel_separation>
       <wheel_diameter>${2 * wheel_radius}</wheel_diameter>
-      <!-- 限制 -->
       <max_wheel_torque>20</max_wheel_torque>
       <max_wheel_acceleration>1.0</max_wheel_acceleration>
-      <!-- 输出 -->
       <publish_odom>true</publish_odom>
       <publish_odom_tf>true</publish_odom_tf>
@@ -25,5 +20,4 @@
     </plugin>
   </gazebo>
-  <!-- Gazebo插件：二维激光雷达 -->
   <gazebo reference="laser_link">
     <material>Gazebo/Red</material>
@@ -62,5 +56,73 @@
     </sensor>
   </gazebo>
-  <!-- Gazebo材质 -->
+  <gazebo reference="imu_link">
+    <material>Gazebo/Green</material>
+    <sensor type="imu" name="imu_sensor">
+      <plugin filename="libgazebo_ros_imu_sensor.so" name="imu_plugin">
+        <ros>
+          <namespace>/</namespace>
+          <remapping>~/out:=imu</remapping>
+        </ros>
+        <initial_orientation_as_reference>false</initial_orientation_as_reference>
+      </plugin>
+      <always_on>true</always_on>
+      <update_rate>100</update_rate>
+      <visualize>true</visualize>
+      <imu>
+        <angular_velocity>
+          <x>
+            <noise type="gaussian">
+              <mean>0.0</mean>
+              <stddev>0.0002</stddev>
+              <bias_mean>0.0</bias_mean>
+              <bias_stddev>0.0</bias_stddev>
+            </noise>
+          </x>
+          <y>
+            <noise type="gaussian">
+              <mean>0.0</mean>
+              <stddev>0.0002</stddev>
+              <bias_mean>0.0</bias_mean>
+              <bias_stddev>0.0</bias_stddev>
+            </noise>
+          </y>
+          <z>
+            <noise type="gaussian">
+              <mean>0.0</mean>
+              <stddev>0.0002</stddev>
+              <bias_mean>0.0</bias_mean>
+              <bias_stddev>0.0</bias_stddev>
+            </noise>
+          </z>
+        </angular_velocity>
+        <linear_acceleration>
+          <x>
+            <noise type="gaussian">
+              <mean>0.0</mean>
+              <stddev>0.01</stddev>
+              <bias_mean>0.0</bias_mean>
+              <bias_stddev>0.0</bias_stddev>
+            </noise>
+          </x>
+          <y>
+            <noise type="gaussian">
+              <mean>0.0</mean>
+              <stddev>0.01</stddev>
+              <bias_mean>0.0</bias_mean>
+              <bias_stddev>0.0</bias_stddev>
+            </noise>
+          </y>
+          <z>
+            <noise type="gaussian">
+              <mean>0.0</mean>
+              <stddev>0.01</stddev>
+              <bias_mean>0.0</bias_mean>
+              <bias_stddev>0.0</bias_stddev>
+            </noise>
+          </z>
+        </linear_acceleration>
+      </imu>
+    </sensor>
+  </gazebo>
   <gazebo reference="base_link">
     <material>Gazebo/Blue</material>
@@ -68,7 +130,28 @@
   <gazebo reference="left_wheel">
     <material>Gazebo/Black</material>
+    <kp>60000.0</kp>
+    <kd>50.0</kd>
+    <mu1>1.0</mu1>
+    <mu2>1.0</mu2>
   </gazebo>
   <gazebo reference="right_wheel">
     <material>Gazebo/Black</material>
+    <kp>60000.0</kp>
+    <kd>50.0</kd>
+    <mu1>1.0</mu1>
+    <mu2>1.0</mu2>
+  </gazebo>
+  <gazebo reference="imu_link">
+    <material>Gazebo/Green</material>
+  </gazebo>
+  <gazebo reference="front_caster">
+    <mu1>0.1</mu1>
+    <mu2>0.2</mu2>
+    <material>Gazebo/Grey</material>
+  </gazebo>
+  <gazebo reference="rear_caster">
+    <mu1>0.0</mu1>
+    <mu2>0.0</mu2>
+    <material>Gazebo/Grey</material>
   </gazebo>
 </robot>
